File: mech.kicad_sch (KiCad schematic)
At the start: 4 parts

Commit message: Resistor networks changed to 0603 'cause JLCPCB has those as 'basic parts' & aunch of tweaks. (WIP)
Parts:
- H1, H2, H3, H4: value MountingHole_Pad -> (none); footprint MountingHole:MountingHole_3.2mm_M3_ISO14580_Pad -> (none)
Changed lines of the file:
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@@
       (effects (font (size 1.27 1.27)) (justify left))
     )
-    (property "Value" "MountingHole_Pad" (id 1) (at 66.04 54.6099 0)
+    (property "Value" "" (id 1) (at 66.04 54.6099 0)
       (effects (font (size 1.27 1.27)) (justify left) hide)
     )
-    (property "Footprint" "MountingHole:MountingHole_3.2mm_M3_ISO14580_Pad" (id 2) (at 63.5 54.61 0)
+    (property "Footprint" "" (id 2) (at 63.5 54.61 0)
       (effects (font (size 1.27 1.27)) hide)
     )
@@
       (effects (font (size 1.27 1.27)) (justify left))
     )
-    (property "Value" "MountingHole_Pad" (id 1) (at 59.69 54.6099 0)
+    (property "Value" "" (id 1) (at 59.69 54.6099 0)
       (effects (font (size 1.27 1.27)) (justify left) hide)
     )
-    (property "Footprint" "MountingHole:MountingHole_3.2mm_M3_ISO14580_Pad" (id 2) (at 57.15 54.61 0)
+    (property "Footprint" "" (id 2) (at 57.15 54.61 0)
       (effects (font (size 1.27 1.27)) hide)
     )
@@
       (effects (font (size 1.27 1.27)) (justify left))
     )
-    (property "Value" "MountingHole_Pad" (id 1) (at 72.39 54.6099 0)
+    (property "Value" "" (id 1) (at 72.39 54.6099 0)
       (effects (font (size 1.27 1.27)) (justify left) hide)
     )
-    (property "Footprint" "MountingHole:MountingHole_3.2mm_M3_ISO14580_Pad" (id 2) (at 69.85 54.61 0)
+    (property "Footprint" "" (id 2) (at 69.85 54.61 0)
       (effects (font (size 1.27 1.27)) hide)
     )
@@
       (effects (font (size 1.27 1.27)) (justify left))
     )
-    (property "Value" "MountingHole_Pad" (id 1) (at 53.34 54.6099 0)
+    (property "Value" "" (id 1) (at 53.34 54.6099 0)
       (effects (font (size 1.27 1.27)) (justify left) hide)
     )
-    (property "Footprint" "MountingHole:MountingHole_3.2mm_M3_ISO14580_Pad" (id 2) (at 50.8 54.61 0)
+    (property "Footprint" "" (id 2) (at 50.8 54.61 0)
       (effects (font (size 1.27 1.27)) hide)
     )

Commit message: temp
Parts:
- H1, H2, H3, H4: value (none) -> MountingHole_Pad
Changed lines of the file:
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@@
       (effects (font (size 1.27 1.27)) (justify left))
     )
-    (property "Value" "" (id 1) (at 66.04 54.6099 0)
+    (property "Value" "MountingHole_Pad" (id 1) (at 66.04 54.6099 0)
       (effects (font (size 1.27 1.27)) (justify left) hide)
     )
@@
       (effects (font (size 1.27 1.27)) (justify left))
     )
-    (property "Value" "" (id 1) (at 59.69 54.6099 0)
+    (property "Value" "MountingHole_Pad" (id 1) (at 59.69 54.6099 0)
       (effects (font (size 1.27 1.27)) (justify left) hide)
     )
@@
       (effects (font (size 1.27 1.27)) (justify left))
     )
-    (property "Value" "" (id 1) (at 72.39 54.6099 0)
+    (property "Value" "MountingHole_Pad" (id 1) (at 72.39 54.6099 0)
       (effects (font (size 1.27 1.27)) (justify left) hide)
     )
@@
       (effects (font (size 1.27 1.27)) (justify left))
     )
-    (property "Value" "" (id 1) (at 53.34 54.6099 0)
+    (property "Value" "MountingHole_Pad" (id 1) (at 53.34 54.6099 0)
       (effects (font (size 1.27 1.27)) (justify left) hide)
     )

Commit message: Removed 'Element14' field from all sch/pcb components
Parts:
- H1, H2, H3, H4: footprint (none) -> MountingHole:MountingHole_3.2mm_M3_ISO14580_Pad
Changed lines of the file:
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@@
       (effects (font (size 1.27 1.27)) (justify left) hide)
     )
-    (property "Footprint" "" (id 2) (at 63.5 54.61 0)
+    (property "Footprint" "MountingHole:MountingHole_3.2mm_M3_ISO14580_Pad" (id 2) (at 63.5 54.61 0)
       (effects (font (size 1.27 1.27)) hide)
     )
@@
       (effects (font (size 1.27 1.27)) (justify left) hide)
     )
-    (property "Footprint" "" (id 2) (at 57.15 54.61 0)
+    (property "Footprint" "MountingHole:MountingHole_3.2mm_M3_ISO14580_Pad" (id 2) (at 57.15 54.61 0)
       (effects (font (size 1.27 1.27)) hide)
     )
@@
       (effects (font (size 1.27 1.27)) (justify left) hide)
     )
-    (property "Footprint" "" (id 2) (at 69.85 54.61 0)
+    (property "Footprint" "MountingHole:MountingHole_3.2mm_M3_ISO14580_Pad" (id 2) (at 69.85 54.61 0)
       (effects (font (size 1.27 1.27)) hide)
     )
@@
       (effects (font (size 1.27 1.27)) (justify left) hide)
     )
-    (property "Footprint" "" (id 2) (at 50.8 54.61 0)
+    (property "Footprint" "MountingHole:MountingHole_3.2mm_M3_ISO14580_Pad" (id 2) (at 50.8 54.61 0)
       (effects (font (size 1.27 1.27)) hide)
     )
