File: mech.kicad_sch (KiCad schematic)
At the start: 4 parts

Commit message: Part supply references wip.
Parts:
- H1, H2, H3, H4: footprint MountingHole:MountingHole_3.2mm_M3_ISO14580_Pad -> (none)
Changed lines of the file:
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@@
       (effects (font (size 1.27 1.27)) (justify left) hide)
     )
-    (property "Footprint" "MountingHole:MountingHole_3.2mm_M3_ISO14580_Pad" (id 2) (at 63.5 54.61 0)
+    (property "Footprint" "" (id 2) (at 63.5 54.61 0)
       (effects (font (size 1.27 1.27)) hide)
     )
@@
       (effects (font (size 1.27 1.27)) (justify left) hide)
     )
-    (property "Footprint" "MountingHole:MountingHole_3.2mm_M3_ISO14580_Pad" (id 2) (at 57.15 54.61 0)
+    (property "Footprint" "" (id 2) (at 57.15 54.61 0)
       (effects (font (size 1.27 1.27)) hide)
     )
@@
       (effects (font (size 1.27 1.27)) (justify left) hide)
     )
-    (property "Footprint" "MountingHole:MountingHole_3.2mm_M3_ISO14580_Pad" (id 2) (at 69.85 54.61 0)
+    (property "Footprint" "" (id 2) (at 69.85 54.61 0)
       (effects (font (size 1.27 1.27)) hide)
     )
@@
       (effects (font (size 1.27 1.27)) (justify left) hide)
     )
-    (property "Footprint" "MountingHole:MountingHole_3.2mm_M3_ISO14580_Pad" (id 2) (at 50.8 54.61 0)
+    (property "Footprint" "" (id 2) (at 50.8 54.61 0)
       (effects (font (size 1.27 1.27)) hide)
     )

Commit message: Completed change to screw terminal blocks. (P16/17 remains JST.)
Parts:
- H1, H2, H3, H4: value MountingHole_Pad -> (none)
Changed lines of the file:
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@@
       (effects (font (size 1.27 1.27)) (justify left))
     )
-    (property "Value" "MountingHole_Pad" (id 1) (at 66.04 54.6099 0)
+    (property "Value" "" (id 1) (at 66.04 54.6099 0)
       (effects (font (size 1.27 1.27)) (justify left) hide)
     )
@@
       (effects (font (size 1.27 1.27)) (justify left))
     )
-    (property "Value" "MountingHole_Pad" (id 1) (at 59.69 54.6099 0)
+    (property "Value" "" (id 1) (at 59.69 54.6099 0)
       (effects (font (size 1.27 1.27)) (justify left) hide)
     )
@@
       (effects (font (size 1.27 1.27)) (justify left))
     )
-    (property "Value" "MountingHole_Pad" (id 1) (at 72.39 54.6099 0)
+    (property "Value" "" (id 1) (at 72.39 54.6099 0)
       (effects (font (size 1.27 1.27)) (justify left) hide)
     )
@@
       (effects (font (size 1.27 1.27)) (justify left))
     )
-    (property "Value" "MountingHole_Pad" (id 1) (at 53.34 54.6099 0)
+    (property "Value" "" (id 1) (at 53.34 54.6099 0)
       (effects (font (size 1.27 1.27)) (justify left) hide)
     )

Commit message: Changed name to Shapeoko LPT Interface v2.0
Parts:
- H1, H2, H3, H4: value (none) -> MountingHole_Pad
Other:
- title: (none) -> Shapeoko LPT Interface — Mechanical
Changed lines of the file:
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@@
   (paper "A4")
   (title_block
-    (date "2022-05-24")
+    (title "Shapeoko LPT Interface — Mechanical")
+    (date "2022-06-02")
     (rev "2.0")
   )
@@
       (effects (font (size 1.27 1.27)) (justify left))
     )
-    (property "Value" "" (id 1) (at 66.04 54.6099 0)
+    (property "Value" "MountingHole_Pad" (id 1) (at 66.04 54.6099 0)
       (effects (font (size 1.27 1.27)) (justify left) hide)
     )
@@
       (effects (font (size 1.27 1.27)) (justify left))
     )
-    (property "Value" "" (id 1) (at 59.69 54.6099 0)
+    (property "Value" "MountingHole_Pad" (id 1) (at 59.69 54.6099 0)
       (effects (font (size 1.27 1.27)) (justify left) hide)
     )
@@
       (effects (font (size 1.27 1.27)) (justify left))
     )
-    (property "Value" "" (id 1) (at 72.39 54.6099 0)
+    (property "Value" "MountingHole_Pad" (id 1) (at 72.39 54.6099 0)
       (effects (font (size 1.27 1.27)) (justify left) hide)
     )
@@
       (effects (font (size 1.27 1.27)) (justify left))
     )
-    (property "Value" "" (id 1) (at 53.34 54.6099 0)
+    (property "Value" "MountingHole_Pad" (id 1) (at 53.34 54.6099 0)
       (effects (font (size 1.27 1.27)) (justify left) hide)
     )

Commit message: Completed element14 part codes
Parts:
- H1, H2, H3, H4: E14MFR# (none) -> DNI; E14MOQ (none) -> 0; E14PART (none) -> DNI; JLCMOQ (none) -> 0; JLCPART (none) -> DNI
Changed lines of the file:
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@@
       (effects (font (size 1.27 1.27)) hide)
     )
-    (property "JLCPART" "" (id 4) (at 63.5 54.61 0)
+    (property "JLCPART" "DNI" (id 4) (at 63.5 54.61 0)
       (effects (font (size 1.27 1.27)) hide)
     )
     (property "JLCMFR#" "DNI" (id 5) (at 63.5 54.61 0)
+      (effects (font (size 1.27 1.27)) hide)
+    )
+    (property "E14MOQ" "0" (id 6) (at 63.5 54.61 0)
+      (effects (font (size 1.27 1.27)) hide)
+    )
+    (property "E14MFR#" "DNI" (id 7) (at 63.5 54.61 0)
+      (effects (font (size 1.27 1.27)) hide)
+    )
+    (property "E14PART" "DNI" (id 8) (at 63.5 54.61 0)
+      (effects (font (size 1.27 1.27)) hide)
+    )
+    (property "JLCMOQ" "0" (id 9) (at 63.5 54.61 0)
       (effects (font (size 1.27 1.27)) hide)
     )
@@
       (effects (font (size 1.27 1.27)) hide)
     )
+    (property "JLCPART" "DNI" (id 6) (at 57.15 54.61 0)
+      (effects (font (size 1.27 1.27)) hide)
+    )
+    (property "E14MOQ" "0" (id 7) (at 57.15 54.61 0)
+      (effects (font (size 1.27 1.27)) hide)
+    )
+    (property "E14MFR#" "DNI" (id 8) (at 57.15 54.61 0)
+      (effects (font (size 1.27 1.27)) hide)
+    )
+    (property "E14PART" "DNI" (id 9) (at 57.15 54.61 0)
+      (effects (font (size 1.27 1.27)) hide)
+    )
+    (property "JLCMOQ" "0" (id 10) (at 57.15 54.61 0)
+      (effects (font (size 1.27 1.27)) hide)
+    )
     (pin "1")
   )
@@
       (effects (font (size 1.27 1.27)) hide)
     )
-    (property "JLCPART" "" (id 4) (at 69.85 54.61 0)
+    (property "JLCPART" "DNI" (id 4) (at 69.85 54.61 0)
       (effects (font (size 1.27 1.27)) hide)
     )
     (property "JLCMFR#" "DNI" (id 5) (at 69.85 54.61 0)
+      (effects (font (size 1.27 1.27)) hide)
+    )
+    (property "E14MOQ" "0" (id 6) (at 69.85 54.61 0)
+      (effects (font (size 1.27 1.27)) hide)
+    )
+    (property "E14MFR#" "DNI" (id 7) (at 69.85 54.61 0)
+      (effects (font (size 1.27 1.27)) hide)
+    )
+    (property "E14PART" "DNI" (id 8) (at 69.85 54.61 0)
+      (effects (font (size 1.27 1.27)) hide)
+    )
+    (property "JLCMOQ" "0" (id 9) (at 69.85 54.61 0)
       (effects (font (size 1.27 1.27)) hide)
     )
@@
       (effects (font (size 1.27 1.27)) hide)
     )
+    (property "JLCPART" "DNI" (id 6) (at 50.8 54.61 0)
+      (effects (font (size 1.27 1.27)) hide)
+    )
+    (property "E14MOQ" "0" (id 7) (at 50.8 54.61 0)
+      (effects (font (size 1.27 1.27)) hide)
+    )
+    (property "E14MFR#" "DNI" (id 8) (at 50.8 54.61 0)
+      (effects (font (size 1.27 1.27)) hide)
+    )
+    (property "E14PART" "DNI" (id 9) (at 50.8 54.61 0)
+      (effects (font (size 1.27 1.27)) hide)
+    )
+    (property "JLCMOQ" "0" (id 10) (at 50.8 54.61 0)
+      (effects (font (size 1.27 1.27)) hide)
+    )

Commit message: Change and reposition JP16/17 connector to screw terminal.
Parts:
- H1, H2, H3, H4: footprint (none) -> MountingHole:MountingHole_3.2mm_M3_ISO14580_Pad
Changed lines of the file:
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@@
       (effects (font (size 1.27 1.27)) (justify left) hide)
     )
-    (property "Footprint" "" (id 2) (at 63.5 54.61 0)
+    (property "Footprint" "MountingHole:MountingHole_3.2mm_M3_ISO14580_Pad" (id 2) (at 63.5 54.61 0)
       (effects (font (size 1.27 1.27)) hide)
     )
@@
       (effects (font (size 1.27 1.27)) (justify left) hide)
     )
-    (property "Footprint" "" (id 2) (at 57.15 54.61 0)
+    (property "Footprint" "MountingHole:MountingHole_3.2mm_M3_ISO14580_Pad" (id 2) (at 57.15 54.61 0)
       (effects (font (size 1.27 1.27)) hide)
     )
@@
       (effects (font (size 1.27 1.27)) (justify left) hide)
     )
-    (property "Footprint" "" (id 2) (at 69.85 54.61 0)
+    (property "Footprint" "MountingHole:MountingHole_3.2mm_M3_ISO14580_Pad" (id 2) (at 69.85 54.61 0)
       (effects (font (size 1.27 1.27)) hide)
     )
@@
       (effects (font (size 1.27 1.27)) (justify left) hide)
     )
-    (property "Footprint" "" (id 2) (at 50.8 54.61 0)
+    (property "Footprint" "MountingHole:MountingHole_3.2mm_M3_ISO14580_Pad" (id 2) (at 50.8 54.61 0)
       (effects (font (size 1.27 1.27)) hide)
     )
