File: controller.kicad_sch (KiCad schematic)
At the start: 3 parts

Commit message: Tweaks and JLCPCB LCSC field name changes.
Parts:
- JP1, JP2, JP3: value 1x02_2.54 -> (none); footprint Connector_PinHeader_2.54mm:PinHeader_1x03_P2.54mm_Vertical -> (none)
Changed lines of the file:
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@@
       (effects (font (size 1.27 1.27)) (justify right))
     )
-    (property "Value" "1x02_2.54" (id 1) (at 165.735 54.61 0)
+    (property "Value" "" (id 1) (at 165.735 54.61 0)
       (effects (font (size 1.27 1.27)) (justify right) hide)
     )
-    (property "Footprint" "Connector_PinHeader_2.54mm:PinHeader_1x03_P2.54mm_Vertical" (id 2) (at 162.56 58.42 0)
+    (property "Footprint" "" (id 2) (at 162.56 58.42 0)
       (effects (font (size 1.27 1.27)) hide)
     )
@@
       (effects (font (size 1.27 1.27)) (justify right))
     )
-    (property "Value" "1x02_2.54" (id 1) (at 167.64 128.905 0)
+    (property "Value" "" (id 1) (at 167.64 128.905 0)
       (effects (font (size 1.27 1.27)) (justify right) hide)
     )
-    (property "Footprint" "Connector_PinHeader_2.54mm:PinHeader_1x03_P2.54mm_Vertical" (id 2) (at 163.83 132.08 0)
+    (property "Footprint" "" (id 2) (at 163.83 132.08 0)
       (effects (font (size 1.27 1.27)) hide)
     )
@@
       (effects (font (size 1.27 1.27)) (justify right))
     )
-    (property "Value" "1x02_2.54" (id 1) (at 160.02 150.495 0)
+    (property "Value" "" (id 1) (at 160.02 150.495 0)
       (effects (font (size 1.27 1.27)) (justify right) hide)
     )
-    (property "Footprint" "Connector_PinHeader_2.54mm:PinHeader_1x03_P2.54mm_Vertical" (id 2) (at 163.83 147.32 0)
+    (property "Footprint" "" (id 2) (at 163.83 147.32 0)
       (effects (font (size 1.27 1.27)) hide)
     )
@@
       (reference "#PWR09") (unit 1) (value "GND") (footprint "")
     )
-    (path "/91071e44-e7cf-47b2-b33b-9fbb68533ee5/351ab4c7-0f1f-439e-95a1-6d3c498a7e3f"
-      (reference "#PWR010") (unit 1) (value "GND") (footprint "")
-    )
     (path "/91071e44-e7cf-47b2-b33b-9fbb68533ee5/87009279-acdb-4b36-a68d-cc578876c759"
       (reference "#PWR011") (unit 1) (value "GND") (footprint "")
@@
     )
     (path "/91071e44-e7cf-47b2-b33b-9fbb68533ee5/344b03d4-3c6c-464c-bdec-ef5b420f9cd5"
-      (reference "R4") (unit 1) (value "100K") (footprint "Resistor_SMD:R_0603_1608Metric")
+      (reference "R4") (unit 1) (value "220K") (footprint "Resistor_SMD:R_0603_1608Metric")
     )
     (path "/91071e44-e7cf-47b2-b33b-9fbb68533ee5/90c4c72f-583b-4f3f-9010-af0e05aa12cf"
@@
     )
     (path "/91071e44-e7cf-47b2-b33b-9fbb68533ee5/ba382702-479e-476c-9107-5221aaf45013"
-      (reference "R8") (unit 1) (value "270K") (footprint "Resistor_SMD:R_0603_1608Metric")
+      (reference "R8") (unit 1) (value "680K") (footprint "Resistor_SMD:R_0603_1608Metric")
     )
     (path "/91071e44-e7cf-47b2-b33b-9fbb68533ee5/3c6161c2-fed7-42c6-b1a9-6d6d6c234632"
-      (reference "R9") (unit 1) (value "270K") (footprint "Resistor_SMD:R_0603_1608Metric")
+      (reference "R9") (unit 1) (value "330K") (footprint "Resistor_SMD:R_0603_1608Metric")
     )
     (path "/91071e44-e7cf-47b2-b33b-9fbb68533ee5/40735455-6a46-469f-906f-764809b4c488"
-      (reference "R10") (unit 1) (value "130K") (footprint "Resistor_SMD:R_0603_1608Metric")
-    )
-    (path "/91071e44-e7cf-47b2-b33b-9fbb68533ee5/811f37f3-39a2-406c-be10-1b20381569fd"
-      (reference "R11") (unit 1) (value "1M") (footprint "Resistor_SMD:R_0603_1608Metric")
+      (reference "R10") (unit 1) (value "100K") (footprint "Resistor_SMD:R_0603_1608Metric")
     )
     (path "/91071e44-e7cf-47b2-b33b-9fbb68533ee5/41a526e6-7b9c-4fee-8d0e-27327ed96432"

Commit message: I'm soooo done with this board! :/
Parts:
- JP1, JP2, JP3: value (none) -> 1x02_2.54; footprint (none) -> Connector_PinHeader_2.54mm:PinHeader_1x03_P2.54mm_Vertical; E14MOQ (none) -> 50; JLCMFR# (none) -> DNI; MOQ 50 -> (none)

Commit message: Some fixes .... and ... a MAJOR fuck up on the power connector, after the board went into production already.
Parts:
- JP1, JP2, JP3: value 1x02_2.54 -> (none); footprint Connector_PinHeader_2.54mm:PinHeader_1x03_P2.54mm_Vertical -> (none)
Changed lines of the file:
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@@
       (effects (font (size 1.27 1.27)) (justify right))
     )
-    (property "Value" "1x02_2.54" (id 1) (at 165.735 54.61 0)
+    (property "Value" "" (id 1) (at 165.735 54.61 0)
       (effects (font (size 1.27 1.27)) (justify right) hide)
     )
-    (property "Footprint" "Connector_PinHeader_2.54mm:PinHeader_1x03_P2.54mm_Vertical" (id 2) (at 162.56 58.42 0)
+    (property "Footprint" "" (id 2) (at 162.56 58.42 0)
       (effects (font (size 1.27 1.27)) hide)
     )
@@
       (effects (font (size 1.27 1.27)) (justify right))
     )
-    (property "Value" "1x02_2.54" (id 1) (at 167.64 128.905 0)
+    (property "Value" "" (id 1) (at 167.64 128.905 0)
       (effects (font (size 1.27 1.27)) (justify right) hide)
     )
-    (property "Footprint" "Connector_PinHeader_2.54mm:PinHeader_1x03_P2.54mm_Vertical" (id 2) (at 163.83 132.08 0)
+    (property "Footprint" "" (id 2) (at 163.83 132.08 0)
       (effects (font (size 1.27 1.27)) hide)
     )
@@
       (effects (font (size 1.27 1.27)) (justify right))
     )
-    (property "Value" "1x02_2.54" (id 1) (at 160.02 150.495 0)
+    (property "Value" "" (id 1) (at 160.02 150.495 0)
       (effects (font (size 1.27 1.27)) (justify right) hide)
     )
-    (property "Footprint" "Connector_PinHeader_2.54mm:PinHeader_1x03_P2.54mm_Vertical" (id 2) (at 163.83 147.32 0)
+    (property "Footprint" "" (id 2) (at 163.83 147.32 0)
       (effects (font (size 1.27 1.27)) hide)
     )
@@
     )
     (path "/96816895-f098-4539-b755-2c649e465f79/90af7ce1-461c-4bca-a8d4-d0cf8ba46de0"
-      (reference "J5") (unit 1) (value "JST_B6B-XH") (footprint "Connector_JST:JST_EH_S6B-EH_1x06_P2.50mm_Horizontal")
+      (reference "J5") (unit 1) (value "JST_S6B-XH") (footprint "Connector_JST:JST_EH_S6B-EH_1x06_P2.50mm_Horizontal")
     )
     (path "/96816895-f098-4539-b755-2c649e465f79/7fdcc566-2de3-4184-aa03-426dc6a88796"
-      (reference "J6") (unit 1) (value "JST_1x04") (footprint "Connector_JST:JST_EH_S4B-EH_1x04_P2.50mm_Horizontal")
+      (reference "J6") (unit 1) (value "JST_S4B-XH") (footprint "Connector_JST:JST_EH_S4B-EH_1x04_P2.50mm_Horizontal")
     )
     (path "/96816895-f098-4539-b755-2c649e465f79/fb128caf-d108-4c02-9b32-7ea342816180"
@@
     )
     (path "/96816895-f098-4539-b755-2c649e465f79/65c0d18d-d829-4325-92eb-05b27fac23d2"
-      (reference "J8") (unit 1) (value "JST_1x04") (footprint "Connector_JST:JST_EH_S4B-EH_1x04_P2.50mm_Horizontal")
+      (reference "J8") (unit 1) (value "JST_S4B-XH") (footprint "Connector_JST:JST_EH_S4B-EH_1x04_P2.50mm_Horizontal")
     )
     (path "/96816895-f098-4539-b755-2c649e465f79/4f281608-903b-4ec0-a893-90c9692af024"
-      (reference "J9") (unit 1) (value "JST_1x04") (footprint "Connector_JST:JST_EH_S4B-EH_1x04_P2.50mm_Horizontal")
+      (reference "J9") (unit 1) (value "JST_S4B-XH") (footprint "Connector_JST:JST_EH_S4B-EH_1x04_P2.50mm_Horizontal")
     )
     (path "/96816895-f098-4539-b755-2c649e465f79/b47f89bb-44a4-4a9f-8b7c-3acd2d90a48a"
@@
     )
     (path "/96816895-f098-4539-b755-2c649e465f79/cdba690a-ad69-489c-88ef-cd1a8ac7b729"
-      (reference "J11") (unit 1) (value "JST_1x04") (footprint "Connector_JST:JST_EH_S4B-EH_1x04_P2.50mm_Horizontal")
+      (reference "J11") (unit 1) (value "JST_S4B-XH") (footprint "Connector_JST:JST_EH_S4B-EH_1x04_P2.50mm_Horizontal")
     )
     (path "/96816895-f098-4539-b755-2c649e465f79/3287a909-8c1d-4161-8291-13ce93b716a3"
@@
     )
     (path "/96816895-f098-4539-b755-2c649e465f79/9859c259-3292-45a3-af2d-b6599b20ac97"
-      (reference "J13") (unit 1) (value "JST_01x02") (footprint "Connector_JST:JST_EH_B2B-EH-A_1x02_P2.50mm_Vertical")
+      (reference "J13") (unit 1) (value "JST_B2B-XH") (footprint "Connector_JST:JST_EH_B2B-EH-A_1x02_P2.50mm_Vertical")
     )
     (path "/96816895-f098-4539-b755-2c649e465f79/bb956b12-f9f1-4980-8383-5ee521965984"
-      (reference "J14") (unit 1) (value "JST_1x02") (footprint "Connector_JST:JST_EH_S2B-EH_1x02_P2.50mm_Horizontal")
+      (reference "J14") (unit 1) (value "JST_S2B-XH") (footprint "Connector_JST:JST_EH_S2B-EH_1x02_P2.50mm_Horizontal")
     )
     (path "/96816895-f098-4539-b755-2c649e465f79/6117399c-16dc-46e8-bf1a-9bba26e70efc"
@@
     )
     (path "/954a9830-ad6d-4d7c-92ee-21f7ecb42ef4/94412c46-f9be-4bc2-ba14-0943a11adc09"
-      (reference "R13") (unit 1) (value "22") (footprint "Resistor_SMD:R_0603_1608Metric")
+      (reference "R13") (unit 1) (value "22R") (footprint "Resistor_SMD:R_0603_1608Metric")
     )
     (path "/954a9830-ad6d-4d7c-92ee-21f7ecb42ef4/9efea078-f3ea-47ef-8d6c-02bb6adceb71"

Commit message: Corrected unbelievably DUMB ballsup on input power connector.
Parts:
- JP1, JP2, JP3: value (none) -> 1x02_2.54; footprint (none) -> Connector_PinHeader_2.54mm:PinHeader_1x03_P2.54mm_Vertical
Changed lines of the file:
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@@
       (effects (font (size 1.27 1.27)) (justify right))
     )
-    (property "Value" "" (id 1) (at 165.735 54.61 0)
+    (property "Value" "1x02_2.54" (id 1) (at 165.735 54.61 0)
       (effects (font (size 1.27 1.27)) (justify right) hide)
     )
-    (property "Footprint" "" (id 2) (at 162.56 58.42 0)
+    (property "Footprint" "Connector_PinHeader_2.54mm:PinHeader_1x03_P2.54mm_Vertical" (id 2) (at 162.56 58.42 0)
       (effects (font (size 1.27 1.27)) hide)
     )
@@
       (effects (font (size 1.27 1.27)) (justify right))
     )
-    (property "Value" "" (id 1) (at 167.64 128.905 0)
+    (property "Value" "1x02_2.54" (id 1) (at 167.64 128.905 0)
       (effects (font (size 1.27 1.27)) (justify right) hide)
     )
-    (property "Footprint" "" (id 2) (at 163.83 132.08 0)
+    (property "Footprint" "Connector_PinHeader_2.54mm:PinHeader_1x03_P2.54mm_Vertical" (id 2) (at 163.83 132.08 0)
       (effects (font (size 1.27 1.27)) hide)
     )
@@
       (effects (font (size 1.27 1.27)) (justify right))
     )
-    (property "Value" "" (id 1) (at 160.02 150.495 0)
+    (property "Value" "1x02_2.54" (id 1) (at 160.02 150.495 0)
       (effects (font (size 1.27 1.27)) (justify right) hide)
     )
-    (property "Footprint" "" (id 2) (at 163.83 147.32 0)
+    (property "Footprint" "Connector_PinHeader_2.54mm:PinHeader_1x03_P2.54mm_Vertical" (id 2) (at 163.83 147.32 0)
       (effects (font (size 1.27 1.27)) hide)
     )
