File: controller.kicad_sch (KiCad schematic)
At the start: 14 parts, among them J1 Conn_01x06_Female, J2 Conn_01x06_Female, J3 Conn_01x022_Male

Commit message: v3.3 WIP
Parts:
- added NT29: NetTie_2, -Project:NetTie-2_SMD_Pad0.3mm, symbol Device:NetTie_2
Connections:
- net GND: now also NT19.1, NT19.2, NT29.2
- net GND1: now also J2.23 (Pin_23); no longer H1.1, H2.1, J1.1 (Pin_1)
- net GND2: now also H1.1, H2.1, J1.1 (Pin_1); no longer J2.23 (Pin_23), NT19.1
- net GNDA: now also NT29.1; no longer NT19.2
Other:
- moved on the sheet: NT19, NT20, NT21
