File: lpt.kicad_sch (KiCad schematic)
At the start: 16 parts, among them J4 DB25 FEMALE, U4 74HC245, U5 74HC245, U6 ACSL-6310, U7 ACSL-6310

Commit message: checkpoint
Parts:
- removed JP1: 1x03_2.54, Connector_PinHeader_2.54mm:PinHeader_1x03_P2.54mm_Vertical, symbol Jumper:Jumper_3_Open
- renumbered C15 to C10, C17 to C11, C16 to C12, C14 to C9, J4 to J6, JP8 to JP3, R19 to R13, RN2 to RN1, RN1 to RN2, U4 to U2, U5 to U3, U7 to U4, U6 to U5
Connections:
- net P10_IN: now also RN3.8 (R1.2); no longer RN4.1 (R1.1)
- net P10_OUT: now also RN1.8 (R1.2), U4.11 (O1); no longer RN2.5 (R4.2), U5.14 (O1)
- net P11_OUT: now also RN1.7 (R2.2); no longer RN1.8 (R1.2)
- net P12_OUT: now also RN1.6 (R3.2); no longer RN1.7 (R2.2)
- net P1_IN: now also R13.1, U3.2 (A0)
- net at RN4.8 (R1.2): no longer U5.2 (C1)
- net at RN3.1 (R1.1): now also U4.7 (A4)
- net EMERG_STOP_IN renamed P15_IN
- net GND renamed GND1
Other:
- note added: "End Stop / Probe GND1 Isolation. Shorted for Shapeoko's active sensors."
- note removed: "End Stop / Probe GND Isolation. Shorted for Shapeoko's active sensors."
