File: lpt.kicad_sch (KiCad schematic)
At the start: 19 parts, among them J7 DB25 FEMALE, U2 74HC245, U3 74HC245, U4 ACSL-6310, U5 ACSL-6310

Commit message: more clean-up
Parts:
- removed RN3: 1Kx4, Resistor_SMD:R_Array_Convex_4x0603, symbol Device:R_Pack04
- added R22: 330, Resistor_SMD:R_0603_1608Metric, symbol Device:R
Connections:
- net +5VA: now also U5.5 (A3), U5.7 (A4)
- net P15_IN: now also R22.2
- net at U5.4 (C2): now also R22.1
- net at RN2.5 (R4.2): now also U5.14 (O1)
- net at RN2.7 (R2.2): now also U5.12 (O1)
- net at RN2.8 (R1.2): now also U5.11 (O1)
- no-connect marks 22 -> 8
Changed lines of the file:
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@@
   (junction (at 161.29 76.2) (diameter 0) (color 0 0 0 0)
   )
+  (junction (at 191.77 95.25) (diameter 0) (color 0 0 0 0)
+  )
   (junction (at 160.02 20.32) (diameter 0) (color 0 0 0 0)
   )
@@
   (junction (at 161.29 96.52) (diameter 0) (color 0 0 0 0)
   )
+  (junction (at 191.77 100.33) (diameter 0) (color 0 0 0 0)
+  )
   (junction (at 158.75 46.99) (diameter 0) (color 0 0 0 0)
   )
@@
   (junction (at 44.45 86.36) (diameter 0) (color 0 0 0 0)
   )
-  (no_connect (at 156.21 87.63))
   (no_connect (at 114.3 46.99))
-  (no_connect (at 168.91 106.68))
   (no_connect (at 189.23 92.71))
-  (no_connect (at 189.23 100.33))
   (no_connect (at 189.23 102.87))
-  (no_connect (at 196.85 97.79))
-  (no_connect (at 196.85 100.33))
   (no_connect (at 114.3 99.06))
-  (no_connect (at 207.01 92.71))
   (no_connect (at 114.3 104.14))
-  (no_connect (at 189.23 105.41))
   (no_connect (at 189.23 107.95))
-  (no_connect (at 158.75 87.63))
-  (no_connect (at 196.85 92.71))
-  (no_connect (at 207.01 100.33))
-  (no_connect (at 207.01 97.79))
-  (no_connect (at 168.91 91.44))
   (no_connect (at 114.3 96.52))
   (no_connect (at 114.3 101.6))
-  (no_connect (at 168.91 101.6))
-  (no_connect (at 163.83 87.63))
   (wire (pts (xy 86.995 111.76) (xy 88.9 111.76))
     (stroke (width 0) (type default) (color 0 0 0 0))
@@
     (stroke (width 0) (type default) (color 0 0 0 0))
   )
-  (wire (pts (xy 194.31 97.79) (xy 189.23 97.79))
-    (stroke (width 0) (type default) (color 0 0 0 0))
-  )
   (wire (pts (xy 86.995 54.61) (xy 88.9 54.61))
     (stroke (width 0) (type default) (color 0 0 0 0))
@@
     (stroke (width 0) (type default) (color 0 0 0 0))
   )
+  (wire (pts (xy 168.91 91.44) (xy 163.83 91.44))
+    (stroke (width 0) (type default) (color 0 0 0 0))
+  )
   (wire (pts (xy 181.61 24.13) (xy 181.61 26.67))
     (stroke (width 0) (type default) (color 0 0 0 0))
@@
     (stroke (width 0) (type default) (color 0 0 0 0))
   )
+  (wire (pts (xy 191.77 100.33) (xy 191.77 95.25))
+    (stroke (width 0) (type default) (color 0 0 0 0))
+  )
   (wire (pts (xy 238.125 75.565) (xy 247.015 75.565))
     (stroke (width 0) (type default) (color 0 0 0 0))
@@
     (stroke (width 0) (type default) (color 0 0 0 0))
   )
-  (wire (pts (xy 194.31 95.25) (xy 194.31 97.79))
+  (wire (pts (xy 189.23 97.79) (xy 197.485 97.79))
     (stroke (width 0) (type default) (color 0 0 0 0))
   )
@@
     (stroke (width 0) (type default) (color 0 0 0 0))
   )
+  (wire (pts (xy 163.83 91.44) (xy 163.83 87.63))
+    (stroke (width 0) (type default) (color 0 0 0 0))
+  )
   (wire (pts (xy 39.37 68.58) (xy 55.88 68.58))
     (stroke (width 0) (type default) (color 0 0 0 0))
@@
     (stroke (width 0) (type default) (color 0 0 0 0))
   )
+  (wire (pts (xy 189.23 100.33) (xy 191.77 100.33))
+    (stroke (width 0) (type default) (color 0 0 0 0))
+  )
   (wire (pts (xy 191.77 40.64) (xy 191.77 35.56))
     (stroke (width 0) (type default) (color 0 0 0 0))
@@
     (stroke (width 0) (type default) (color 0 0 0 0))
   )
+  (wire (pts (xy 168.91 101.6) (xy 158.75 101.6))
+    (stroke (width 0) (type default) (color 0 0 0 0))
+  )
   (wire (pts (xy 161.29 87.63) (xy 161.29 96.52))
     (stroke (width 0) (type default) (color 0 0 0 0))
   )
+  (wire (pts (xy 168.91 106.68) (xy 156.21 106.68))
+    (stroke (width 0) (type default) (color 0 0 0 0))
+  )
   (wire (pts (xy 191.77 26.67) (xy 181.61 26.67))
     (stroke (width 0) (type default) (color 0 0 0 0))
@@
     (stroke (width 0) (type default) (color 0 0 0 0))
   )
+  (wire (pts (xy 158.75 101.6) (xy 158.75 87.63))
+    (stroke (width 0) (type default) (color 0 0 0 0))
+  )
   (wire (pts (xy 156.21 21.59) (xy 158.75 21.59))
     (stroke (width 0) (type default) (color 0 0 0 0))
@@
     (stroke (width 0) (type default) (color 0 0 0 0))
   )
+  (wire (pts (xy 191.77 105.41) (xy 191.77 100.33))
+    (stroke (width 0) (type default) (color 0 0 0 0))
+  )
   (wire (pts (xy 44.45 71.12) (xy 44.45 76.2))
     (stroke (width 0) (type default) (color 0 0 0 0))
@@
     (stroke (width 0) (type default) (color 0 0 0 0))
   )
-  (wire (pts (xy 207.01 95.25) (xy 209.55 95.25))
+  (wire (pts (xy 189.23 105.41) (xy 191.77 105.41))
     (stroke (width 0) (type default) (color 0 0 0 0))
   )
@@
     (stroke (width 0) (type default) (color 0 0 0 0))
   )
+  (wire (pts (xy 205.105 97.79) (xy 207.01 97.79))
+    (stroke (width 0) (type default) (color 0 0 0 0))
+  )
   (wire (pts (xy 69.215 140.335) (xy 69.215 139.065))
     (stroke (width 0) (type default) (color 0 0 0 0))
@@
     (stroke (width 0) (type default) (color 0 0 0 0))
   )
+  (wire (pts (xy 156.21 106.68) (xy 156.21 87.63))
+    (stroke (width 0) (type default) (color 0 0 0 0))
+  )
   (wire (pts (xy 88.9 96.52) (xy 88.9 99.06))
     (stroke (width 0) (type default) (color 0 0 0 0))
@@
   )
   (wire (pts (xy 39.37 81.28) (xy 44.45 81.28))
-    (stroke (width 0) (type default) (color 0 0 0 0))
-  )
-  (wire (pts (xy 196.85 95.25) (xy 194.31 95.25))
     (stroke (width 0) (type default) (color 0 0 0 0))
   )
@@
     (effects (font (size 1.27 1.27)) (justify left bottom))
   )
-  (text "open collector\noutputs" (at 125.73 101.6 0)
+  (text "open collector\noutputs" (at 156.845 65.405 0)
     (effects (font (size 1.27 1.27)) (justify left bottom))
   )
@@
     (effects (font (size 1.27 1.27)) (justify left))
   )
-  (hierarchical_label "P15_IN" (shape input) (at 209.55 95.25 0)
+  (hierarchical_label "P15_IN" (shape input) (at 207.01 97.79 0)
     (effects (font (size 1.27 1.27)) (justify left))
   )
@@
     )
     (pin "1")
-  )
-  (symbol (lib_id "Device:R_Pack04") (at 201.93 97.79 90) (mirror x) (unit 1)
-    (in_bom yes) (on_board yes)
-    (property "Reference" "RN3" (id 0) (at 203.835 89.535 90)
-      (effects (font (size 1.27 1.27)) (justify left))
-    )
-    (property "Value" "1Kx4" (id 1) (at 204.47 104.14 90)
-      (effects (font (size 1.27 1.27)) (justify left))
-    )
-    (property "Footprint" "Resistor_SMD:R_Array_Convex_4x0603" (id 2) (at 201.93 104.775 90)
-      (effects (font (size 1.27 1.27)) hide)
-    )
-    (property "Datasheet" "~" (id 3) (at 201.93 97.79 0)
-      (effects (font (size 1.27 1.27)) hide)
-    )
-    (property "E14MOQ" "10" (id 7) (at 201.93 97.79 0)
-      (effects (font (size 1.27 1.27)) hide)
-    )
-    (property "LCSC" "" (id 8) (at 201.93 97.79 0)
-      (effects (font (size 1.27 1.27)) hide)
-    )
-    (property "LCSCMFR#" "" (id 9) (at 201.93 97.79 0)
-      (effects (font (size 1.27 1.27)) hide)
-    )
-    (property "JLCMFR#" "4D03WGJ0102T5E" (id 10) (at 201.93 97.79 0)
-      (effects (font (size 1.27 1.27)) hide)
-    )
-    (property "JLCPART" "C20197" (id 11) (at 201.93 97.79 0)
-      (effects (font (size 1.27 1.27)) hide)
-    )
-    (property "JLCMOQ" "20" (id 12) (at 201.93 97.79 0)
-      (effects (font (size 1.27 1.27)) hide)
-    )
-    (property "E14MFR#" "MP005637" (id 13) (at 201.93 97.79 0)
-      (effects (font (size 1.27 1.27)) hide)
-    )
-    (property "E14PART" "3550064" (id 14) (at 201.93 97.79 0)
-      (effects (font (size 1.27 1.27)) hide)
-    )
-    (pin "1")
-    (pin "2")
-    (pin "3")
-    (pin "4")
-    (pin "5")
-    (pin "6")
-    (pin "7")
-    (pin "8")
   )
   (symbol (lib_id "power:+5VA") (at 196.215 74.295 0) (unit 1)
@@
     (pin "9")
   )
+  (symbol (lib_id "Device:R") (at 201.295 97.79 90) (unit 1)
+    (in_bom yes) (on_board yes)
+    (property "Reference" "R22" (id 0) (at 201.295 95.885 90))
+    (property "Value" "330" (id 1) (at 201.295 97.79 90))
+    (property "Footprint" "Resistor_SMD:R_0603_1608Metric" (id 2) (at 201.295 99.568 90)
+      (effects (font (size 1.27 1.27)) hide)
+    )
+    (property "Datasheet" "~" (id 3) (at 201.295 97.79 0)
+      (effects (font (size 1.27 1.27)) hide)
+    )
+    (property "E14MOQ" "10" (id 5) (at 201.295 97.79 0)
+      (effects (font (size 1.27 1.27)) hide)
+    )
+    (property "E14PART" "1469820" (id 6) (at 201.295 97.79 0)
+      (effects (font (size 1.27 1.27)) hide)
+    )
+    (property "JLCMFR#" "0603WAF5601T5E" (id 7) (at 201.295 97.79 0)
+      (effects (font (size 1.27 1.27)) hide)
+    )
+    (property "JLCMOQ" "20" (id 8) (at 201.295 97.79 0)
+      (effects (font (size 1.27 1.27)) hide)
+    )
+    (property "JLCPART" "C23189" (id 9) (at 201.295 97.79 0)
+      (effects (font (size 1.27 1.27)) hide)
+    )
+    (property "E14MFR#" "CRCW06035K60FKEA" (id 10) (at 201.295 97.79 0)
+      (effects (font (size 1.27 1.27)) hide)
+    )
+    (property "Marking" "331" (id 11) (at 196.85 99.06 90)
+      (effects (font (size 1 1)))
+    )
+    (pin "1")
+    (pin "2")
+  )
   (symbol (lib_id "Device:R") (at 201.93 43.18 90) (unit 1)
