File: controller.kicad_pcb (KiCad board)
At the start: 2 copper layers, 229.8 x 162 mm, 90 parts, among them J1 Conn_01x06_Female, J10 Phoenix MPT, J11 MicroFit_2x04, J12 Phoenix MPT, J13 MicroFit_2x04, J14 Phoenix MPT, J15 JST_B2B-XH, J16 MicroFit_2x04, J17 MLX_1x03, J18 MLX_1x03, J19 Phoenix MPT, J2 Conn_01x022_Male, J3 KYCON_KPJX-4S-S, J4 MicroFit_2x02, J5 24V/5A OUT, J6 DB25 FEMALE, J7 Phoenix MPT, J9 Phoenix MPT, K1 OJS-SH-124HMF, Q1 BC847, Q2 IRFR5305TRPBF, Q3 BC857, Q4 BC847, Q5 BC857, U1 MAX5035BUSA, U2 74HC245, U3 74HC245, U4 ACSL-6310, U5 ACSL-6310

Commit message: checkpoint
Parts:
- moved NT35 4.25 mm to (122.2, 74.3)
- moved J17 3.00 mm to (105.5, 77.9)
- moved J18 3.00 mm to (105.5, 87.5)
- moved JP3 3.00 mm to (98.6, 33.0)
- moved J11 2.99 mm to (98.1, 42.0)
- moved J13 2.99 mm to (98.1, 60.9)
- moved J16 2.99 mm to (98.1, 79.7)
- moved JP1 0.48 mm to (92.3, 97.6)
Routing:
- net /Connectors & Jumpers/PROBE_OUT: track 49.0 -> 43.0 mm
- net GND: track 36.4 -> 30.8 mm, vias 272 -> 295
- net /Connectors & Jumpers/XMIN_OUT: track 42.4 -> 38.7 mm
- net +5V: track 231.0 -> 227.8 mm
- net /Connectors & Jumpers/YMIN_OUT: track 18.7 -> 15.7 mm
- net /Connectors & Jumpers/ZCLK_IN: track 54.8 -> 53.2 mm
- net /Connectors & Jumpers/ZMIN_OUT: track 17.2 -> 15.9 mm
- net /Connectors & Jumpers/YDIR_IN: track 40.4 -> 39.4 mm
- net /Connectors & Jumpers/RELAY4: track 44.6 -> 43.7 mm
- net /Connectors & Jumpers/EN_IN: track 75.0 -> 74.3 mm
- net /Connectors & Jumpers/RELAY1: track 3.75 -> 4.27 mm
- net GNDA: vias 5 -> 37

Commit message: checkpoint
Parts:
- moved JP2 0.85 mm to (88.7, 75.2)
- moved JP6 0.85 mm to (88.7, 56.9)
- moved JP7 0.85 mm to (88.7, 66.7)
Routing:
- net /Connectors & Jumpers/P17_IN: track 8.51 -> 6.41 mm
- net /Connectors & Jumpers/ZDIR_IN: track 58.0 -> 57.0 mm
- net /Connectors & Jumpers/P16_IN: track 6.84 -> 5.91 mm
- net Net-(JP6-Pad3): track 16.1 -> 15.2 mm
- net /Connectors & Jumpers/X_P17_OUT: track 67.0 -> 66.2 mm
- net /Connectors & Jumpers/P1_IN: track 5.51 -> 4.66 mm
- net GND: track 30.8 -> 30.7 mm, vias 295 -> 303

Commit message: checkpoint
Parts:
- moved H1 0.50 mm to (53.5, 119.5)
- moved H2 0.50 mm to (53.5, 188.5)
Changed lines of the file:
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@@
   )
   (footprint "MountingHole:MountingHole_3.2mm_M3_ISO14580_Pad" (layer "F.Cu")
-    (at 53.5 120)
+    (at 53.5 119.5)
     (descr "Mounting Hole 3.2mm, M3, ISO14580")
     (tags "mounting hole 3.2mm m3 iso14580")
@@
   )
   (footprint "MountingHole:MountingHole_3.2mm_M3_ISO14580_Pad" (layer "F.Cu")
-    (at 53.5 188)
+    (at 53.5 188.5)
     (descr "Mounting Hole 3.2mm, M3, ISO14580")
     (tags "mounting hole 3.2mm m3 iso14580")

Commit message: checkpoint
Parts:
- added REF**: MountingHole_3.2mm_M3_ISO14580, MountingHole:MountingHole_3.2mm_M3_ISO14580, F.Cu at (115.3, 30.9)
Other:
- board size 229.8 x 162 mm -> 229.8 x 163.9 mm
Changed lines of the file:
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@@
     )
   )
+  (footprint "MountingHole:MountingHole_3.2mm_M3_ISO14580" (layer "F.Cu")
+    (at 115.34 30.85)
+    (descr "Mounting Hole 3.2mm, no annular, M3, ISO14580")
+    (tags "mounting hole 3.2mm no annular m3 iso14580")
+    (attr exclude_from_pos_files exclude_from_bom)
+    (fp_text reference "REF**" (at 0 -3.75) (layer "F.SilkS")
+      (effects (font (size 1 1) (thickness 0.15)))
+    )
+    (fp_text value "MountingHole_3.2mm_M3_ISO14580" (at 0 3.75) (layer "F.Fab")
+      (effects (font (size 1 1) (thickness 0.15)))
+    )
+    (fp_text user "${REFERENCE}" (at 0 0) (layer "F.Fab")
+      (effects (font (size 1 1) (thickness 0.15)))
+    )
+    (fp_circle (center 0 0) (end 2.75 0) (layer "Cmts.User") (width 0.15) (fill none))
+    (fp_circle (center 0 0) (end 3 0) (layer "F.CrtYd") (width 0.05) (fill none))
+    (pad "" np_thru_hole circle (at 0 0) (size 3.2 3.2) (drill 3.2) (layers *.Cu *.Mask))
+  )
   (footprint "-Project:NetTie-2_SMD_Pad0.3mm" (layer "F.Cu")
     (at 122.225 74.3 -90)
@@
   (gr_line (start 33.489518 68) (end 37.389518 68) (layer "Dwgs.User") (width 0.15))
   (gr_line (start 47.25 95.55) (end 47.3 109.8) (layer "Dwgs.User") (width 0.15))
+  (gr_arc (start 112.868285 29.582061) (mid 112.56029 29.891697) (end 112.137199 30) (layer "Edge.Cuts") (width 0.1))
   (gr_arc (start 37.2 94.507107) (mid 36.492893 94.214214) (end 36.2 93.507107) (layer "Edge.Cuts") (width 0.1))
+  (gr_arc (start 118.54 30) (mid 118.038014 29.819431) (end 117.693566 29.412061) (layer "Edge.Cuts") (width 0.1))
   (gr_line (start 85.9 191) (end 85.9 117) (layer "Edge.Cuts") (width 0.1))
   (gr_arc (start 266 105) (mid 265.707107 105.707107) (end 265 106) (layer "Edge.Cuts") (width 0.1))
@@
   (gr_line (start 36.2 93.507107) (end 36.2 76.007107) (layer "Edge.Cuts") (width 0.1))
   (gr_line (start 37.2 94.507107) (end 49 94.5) (layer "Edge.Cuts") (width 0.1))
+  (gr_line (start 118.54 30) (end 265 30) (layer "Edge.Cuts") (width 0.1))
   (gr_arc (start 51 106) (mid 50.292893 105.707107) (end 50 105) (layer "Edge.Cuts") (width 0.1))
   (gr_arc (start 36.2 76.007107) (mid 36.492893 75.3) (end 37.2 75.007107) (layer "Edge.Cuts") (width 0.1))
@@
   (gr_arc (start 51 192) (mid 50.292893 191.707107) (end 50 191) (layer "Edge.Cuts") (width 0.1))
   (gr_line (start 49 42) (end 37.2 42.007107) (layer "Edge.Cuts") (width 0.1))
+  (gr_arc (start 112.868285 29.582061) (mid 115.231851 28.104121) (end 117.693566 29.412061) (layer "Edge.Cuts") (width 0.1))
   (gr_arc (start 49 94.5) (mid 49.707107 94.792893) (end 50 95.5) (layer "Edge.Cuts") (width 0.1))
   (gr_line (start 84.9 116) (end 51 116) (layer "Edge.Cuts") (width 0.1))
@@
   (gr_arc (start 47.5 74) (mid 47.207107 74.707107) (end 46.5 75) (layer "Edge.Cuts") (width 0.1))
   (gr_arc (start 265 30) (mid 265.707107 30.292893) (end 266 31) (layer "Edge.Cuts") (width 0.1))
-  (gr_line (start 51 30) (end 265 30) (layer "Edge.Cuts") (width 0.1))
+  (gr_line (start 51 30) (end 112.137199 30) (layer "Edge.Cuts") (width 0.1))
   (gr_arc (start 37.2 57.007107) (mid 36.492893 56.714214) (end 36.2 56.007107) (layer "Edge.Cuts") (width 0.1))
   (gr_line (start 81.3 59.5) (end 81.3 60) (layer "F.Fab") (width 0.1))
@@
     (style (thickness 0.15) (arrow_length 1.27) (text_position_mode 2) (extension_height 0.58642) (extension_offset 0.5) keep_text_aligned)
   )
+  (dimension (type orthogonal) (layer "User.1")
+    (pts (xy 50 27.1) (xy 115.34 27.49))
+    (height -3.5)
+    (orientation 0)
+    (gr_text "65.3400 mm" (at 109.44 22.01) (layer "User.1")
+      (effects (font (size 1 1) (thickness 0.15)))
+    )
+    (format (units 3) (units_format 1) (precision 4))
+    (style (thickness 0.15) (arrow_length 1.27) (text_position_mode 2) (extension_height 0.58642) (extension_offset 0.5) keep_text_aligned)
+  )
   (segment (start 87.075 95.3) (end 88.6 93.775) (width 0.3) (layer "F.Cu") (net 1))
   (segment (start 86.35 94.85) (end 86.8 95.3) (width 0.3) (layer "F.Cu") (net 1))
@@
   (via (at 86 91.1) (size 0.7) (drill 0.3) (layers "F.Cu" "B.Cu") (net 3))
   (via (at 88.6 86.7) (size 0.7) (drill 0.3) (layers "F.Cu" "B.Cu") (free) (net 3))
-  (via (at 106.7 30.7) (size 0.7) (drill 0.3) (layers "F.Cu" "B.Cu") (free) (net 3))
+  (via (at 111.87 30.71) (size 0.7) (drill 0.3) (layers "F.Cu" "B.Cu") (free) (net 3))
   (via (at 67.1 95.2) (size 0.7) (drill 0.3) (layers "F.Cu" "B.Cu") (free) (net 3))
   (via (at 123.2 72.175) (size 0.7) (drill 0.3) (layers "F.Cu" "B.Cu") (free) (net 3))
@@
   (via (at 74.225 94.525) (size 0.7) (drill 0.3) (layers "F.Cu" "B.Cu") (free) (net 3))
   (via (at 74.775 69.025) (size 0.7) (drill 0.3) (layers "F.Cu" "B.Cu") (free) (net 3))
-  (via (at 117 30.7) (size 0.7) (drill 0.3) (layers "F.Cu" "B.Cu") (free) (net 3))
+  (via (at 118.76 30.71) (size 0.7) (drill 0.3) (layers "F.Cu" "B.Cu") (free) (net 3))
   (via (at 74.124093 84.952716) (size 0.7) (drill 0.3) (layers "F.Cu" "B.Cu") (free) (net 3))
   (via (at 82.55 61.1) (size 0.7) (drill 0.3) (layers "F.Cu" "B.Cu") (free) (net 3))
@@
     (polygon
       (pts
-        (xy 146.269305 29.769842)
-        (xy 146.370028 105.869842)
-        (xy 35.800032 105.900024)
-        (xy 35.799309 29.900024)
+        (xy 146.265704 26.715087)
+        (xy 146.371321 110.601437)
+        (xy 35.801325 110.631619)
+        (xy 35.795708 26.845269)
       )
     )
@@
     (polygon
       (pts
-        (xy 266.2 30.05)
-        (xy 266.2 106.05)
-        (xy 50 106.05)
+        (xy 266.200104 26.360134)
+        (xy 266.2 110.5)
+        (xy 50 110.5)
         (xy 50 95.6)
         (xy 49 94.5)
@@
         (xy 49.1 41.8)
         (xy 50 40.3)
-        (xy 50 30.043883)
+        (xy 50.000104 26.354017)
       )
     )

Commit message: checkpoint
Parts:
- removed H4, H5: MountingHole_Pad, MountingHole:MountingHole_3.2mm_M3_ISO14580_Pad
- removed REF**: MountingHole_3.2mm_M3_ISO14580, MountingHole:MountingHole_3.2mm_M3_ISO14580
- moved J5 3.50 mm to (119.0, 93.4)
- moved JP4 1.10 mm to (110.7, 42.2)
- moved JP5 0.80 mm to (110.7, 55.2)
- moved NT37 0.80 mm to (107.4, 56.8)
- moved J10 0.60 mm to (120.2, 35.3)
- moved JP8 0.50 mm to (110.7, 68.4)
- moved J12 0.30 mm to (120.2, 48.3)
- moved NT35 0.22 mm to (122.0, 74.3)
Routing:
- net GND1: track 8.87 -> 29.9 mm, vias 6 -> 100
- net 24V_SAFE: track 126.9 -> 128.4 mm
- net /Connectors & Jumpers/EN_IN: track 74.3 -> 73.2 mm
- net GND2: track 5.75 -> 6.52 mm, vias 4 -> 40
- net /Connectors & Jumpers/ZCLK_IN: track 53.3 -> 54.0 mm
- net /Connectors & Jumpers/XDIR_IN: track 39.5 -> 40.1 mm
- net /Connectors & Jumpers/XCLK_IN: track 39.9 -> 40.6 mm
- net /Connectors & Jumpers/YDIR_IN: track 39.4 -> 39.9 mm
- net +5VA: track 176.0 -> 175.5 mm
- net GND: vias 303 -> 300
- added copper zone on F.Cu, net GND1
- added copper zone on F.Cu, net GND2
Other:
- board size 229.8 x 163.9 mm -> 87.3 x 162 mm

Commit message: checkpoint
Parts:
- J5: footprint TerminalBlock_RND:TerminalBlock_RND_205-00232_1x02_P5.08mm_Horizontal -> TerminalBlock_Phoenix:TerminalBlock_Phoenix_MKDS-1,5-2-5.08_1x02_P5.08mm_Horizontal
- moved J5 5.10 mm to (118.7, 98.5), turned to 90 degrees
- renumbered H6 to H4
Connections:
- J5 pad 1: 24V_SAFE -> GND
- J5 pad 2: GND -> 24V_SAFE
Routing:
- net GND: vias 300 -> 303
Other:
- board text added: "+24V"
- board text added: "22"
- board text added: "5A"
- board text added: "AUX"
- board text added: "PWM 5V"
- board text added: "SPINDLE"
- board text added: "github.com/gruvin/shapeoko-lpt"
- board text removed: "*JP2 *JP3"
- board text removed: "+24V 5A"
- board text removed: "6A MAX"
- board text removed: "AGND"
- board text removed: "DGND"
- board text removed: "P1"
- board text removed: "RLY1"
- board text removed: "RLY4"
- board text removed: "VFD"
- board text removed: "https://github.com/gruvin/shapeoko-lpt"

Commit message: MILESTONE: Shrinkage Tk II
Parts:
- removed TH3: JLC_ToolingHole, -Project:JLC_ToolingHole
- moved Q4 18.5 mm to (80.0, 65.0), turned to -90 degrees
- moved R15 16.7 mm to (80.0, 61.4)
- moved D11 15.2 mm to (77.2, 64.7), turned to -90 degrees
- moved R16 14.8 mm to (77.4, 58.1)
- moved Q5 14.8 mm to (77.4, 61.0)
- moved R14 14.6 mm to (81.6, 61.4), turned to 90 degrees
- moved K1 12.2 mm to (78.1, 44.9), turned to 180 degrees
- moved J6 11.1 mm to (69.3, 137.4)
- moved H1 11.1 mm to (64.6, 119.5)
- moved H2 11.1 mm to (64.6, 188.5)
- moved J3 11.1 mm to (69.2, 65.0)
- moved J7 11.0 mm to (51.2, 77.4)
- moved H3 11.0 mm to (64.5, 33.5)
- moved H4 11.0 mm to (64.5, 102.5)
- moved J15 11.0 mm to (51.2, 84.1)
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Connections:
- K1 pad 3: /Connectors & Jumpers/VFD_FWD -> /Connectors & Jumpers/VFD_XGND
- K1 pad 5: /Connectors & Jumpers/VFD_XGND -> /Connectors & Jumpers/VFD_FWD
Routing:
- net +5V: track 227.4 -> 183.9 mm, vias 5 -> 2
- net /Connectors & Jumpers/VFD_FWD: track 47.2 -> 16.5 mm, vias 1 -> 0
- net /Connectors & Jumpers/VFD_XGND: track 39.0 -> 11.8 mm, vias 1 -> 0
- net /LPT Interface/P7_IN: track 24.4 -> 3.73 mm
- net /LPT Interface/P6_IN: track 22.6 -> 2.15 mm
- net /LPT Interface/P15_OUT: track 28.5 -> 8.61 mm
- net /LPT Interface/P5_IN: track 20.7 -> 1.59 mm
- net /Connectors & Jumpers/X_P16_OUT: track 82.4 -> 63.7 mm, vias 3 -> 2
- net /Power/Q1_C: track 74.6 -> 56.9 mm, vias 2 -> 4
- net /LPT Interface/P4_IN: track 17.7 -> 1.12 mm
- net /LPT Interface/P16_IN: track 39.1 -> 22.8 mm
- net /Connectors & Jumpers/X_P17_OUT: track 66.2 -> 50.3 mm
- net /LPT Interface/P3_IN: track 16.0 -> 0.65 mm
- net /LPT Interface/P9_IN: track 18.4 -> 3.34 mm
- net Net-(D11-Pad1): track 7.68 -> 21.3 mm
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- added copper zone on F.Cu, net 24V_SAFE
Other:
- board size 87.3 x 162 mm -> 76.3 x 162 mm
- board text removed: "AUX"
- board text removed: "C.P."
- board text removed: "ESTP"
- board text removed: "P16"
- board text removed: "P17"
- board text removed: "RL4 *"
