File: controller-v3.2.kicad_pcb (KiCad board)
At the start: 2 copper layers, 101.3 x 162.9 mm, 100 parts, among them J1 Conn_01x06_Female, J10 Phoenix MPT, J11 Phoenix MPT, J12 MicroFit_2x04, J13 Phoenix MPT, J14 MicroFit_2x04, J15 JST_B2B-XH, J16 Phoenix MPT, J17 MicroFit_2x04, J18 MLX_1x03, J19 MLX_1x03, J2 Conn_01x06_Female, J20 Phoenix MPT, J3 Conn_01x022_Male, J4 KYCON_KPJX-4S-S, J5 MicroFit_2x02, J6 24V/5A OUT, J7 DB25 FEMALE, J8 Phoenix MPT, K1 OJS-SH-124HMF, Q1 BC847, Q2 FDD5614P, Q3 BC857, Q4 BC847, Q5 BC857, U1 MAX5035BUSA, U2 74HC245, U3 74HC245, U4 ACSL-6310, U5 ACSL-6310, U6 USBLC6-2SC6, U7 ADUM4160, U8 ATmega16U2-A, U9 ATmega328P-A

Commit message: GRBL PCB controller work
Parts:
- moved U6 38.1 mm to (111.3, 139.4)
- moved U7 35.7 mm to (121.4, 134.3)
- moved U8 10.9 mm to (129.1, 180.0)
- moved U9 6.87 mm to (126.5, 154.6)
