File: grbl-interface.kicad_sch (KiCad schematic)
At the start: 42 parts, among them J21 USB_B_Mini, J22 uISP, J23 ISP, SW3 RESET, U6 USBLC6-2SC6, U7 ATmega16U2-A, U8 ADUM4160, U9 ATmega328P-AU, Y1 Crystal_SMD_WE_CFPX-104-4Pin_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, Y2 CSTCE16M0V53-R0 16MHZ

Commit message: MILESTONE — GRBL 1st Draft DRC passses
Parts:
- Y2: footprint (none) -> Crystal:Crystal_SMD_WE_CFPX-104-4Pin_5.0x3.2mm
Changed lines of the file:
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@@
 			)
 		)
-		(property "Footprint" ""
+		(property "Footprint" "Crystal:Crystal_SMD_WE_CFPX-104-4Pin_5.0x3.2mm"
 			(at 176.53 116.84 0)
 			(hide yes)

Commit message: Silkscreen and clearances (mostly)
Parts:
- C28: value TBD_SPACER (DNI) -> ISOLATION approx. 1.5mm (DNI)
- U7: footprint Package_QFP:TQFP-32_7x7mm_P0.8mm -> Package_DFN_QFN:VQFN-32-1EP_4x4mm_P0.4mm_EP2.8x2.8mm
Connections:
- net +5VA: now also C28.1, U8.16 (VBUS2); no longer U8.12 (PIN), U8.13 (SPD), U8.14 (VDD2)
- net GND2: now also C19.2; no longer C19.1
- net VBUS: now also C28.2, U8.1 (VBUS1); no longer U8.3 (VDD1), U8.4 (PDEN), U8.5 (SPU)
- new net: C19.1, U8.12 (PIN), U8.13 (SPD), U8.14 (VDD2)
- new net: C18.2, U8.3 (VDD1), U8.4 (PDEN), U8.5 (SPU)
- no-connect marks 19 -> 20
Other:
- moved on the sheet: C17, C18, C19, R24
